Commit message: Add steering angles, Inertia and fix collapsing arm

File: URDF/testRobot.urdf (robot description, URDF)
Before this commit: robot simplerobot, 6 links, 5 joints
Links:
- link base_link: mass 50.0 -> 40.0

Commit message: self collision avoidance and obstacles

File: URDF/testRobot.urdf (robot description, URDF)
Before this commit: robot simplerobot, 6 links, 5 joints
Links:
- link base_link: mass 40.0 -> 30.0; geometry collision cylinder length=0.4 radius=0.4; visual cylinder length=0.6 radius=0.4
Joints:
- joint arm_1_to_arm_2: limit lower=-1.7 upper=1.7 effort=1000.0 velocity=0.5 -> lower=-2.1 upper=2.1 effort=1000.0 velocity=0.5; origin xyz=0 0 0.7 -> xyz=0 0 0.75
- joint base_to_arm_1: limit lower=-1.7 upper=1.7 effort=1000.0 velocity=0.5 -> lower=-1.8 upper=1.8 effort=1000.0 velocity=0.5; origin xyz=0 0 0.35 -> xyz=0 0 0.5
